Commit message: New version - Wrist working
wrist rotation working and code is lighter

File: actual_arm_urdf.urdf (robot description, URDF)
Before this commit: robot robotic_arm, 6 links, 5 joints
Links:
- added link finger_left; visual box size=0.05 0.02 0.025
- added link finger_right; visual box size=0.05 0.02 0.025
- added link world
Joints:
- added joint finger_left_joint: type prismatic, parent gripper, child finger_left, origin xyz=0 0 0 rpy=0 0 0, axis -1 0 0, limit lower=0 upper=0.04
- added joint finger_right_joint: type prismatic, parent gripper, child finger_right, origin xyz=0 0 0 rpy=0 0 0, axis 1 0 0, limit lower=0 upper=0.04
- added joint world_to_base: type fixed, parent world, child base_link, origin xyz=0 0 0 rpy=0 0 0

Commit message: .

File: actual_arm_urdf.urdf (robot description, URDF)
Before this commit: robot robotic_arm, 9 links, 8 joints
Links:
- link finger_left: geometry visual box size=0.08 0.02 0.03
- link finger_right: geometry visual box size=0.08 0.02 0.03
Joints:
- joint finger_left_joint: axis -1 0 0 -> 0 1 0; limit lower=0 upper=0.04 -> lower=0 upper=1.0; origin xyz=0 0 0 rpy=0 0 0 -> xyz=-0.06 0.025 0 rpy=0 0 0; type prismatic -> revolute
- joint finger_right_joint: axis 1 0 0 -> 0 -1 0; limit lower=0 upper=0.04 -> lower=0 upper=1.0; mimic (none) -> joint=finger_left_joint multiplier=1; origin xyz=0 0 0 rpy=0 0 0 -> xyz=-0.06 -0.025 0 rpy=0 0 0; type prismatic -> revolute

Commit message: 3/4 gpt improvments
3/4 gpt improvments

File: actual_arm_urdf.urdf (robot description, URDF)
Before this commit: robot robotic_arm, 9 links, 8 joints
Joints:
- joint finger_left_joint: axis 0 1 0 -> 1 0 0; limit lower=0 upper=1.0 -> lower=0.0 upper=0.04 effort=1 velocity=0.1; type revolute -> prismatic
- joint finger_right_joint: axis 0 -1 0 -> 1 0 0; limit lower=0 upper=1.0 -> lower=0.0 upper=0.04 effort=1 velocity=0.1; type revolute -> prismatic
