Commit message: integrated IK to move the arm successfully, added requirements.txt, updated the arm urdf according to the arm's physical range, updated the Arduino code to work with IK

File: Hardware/.ipynb_checkpoints/actual_arm_urdf-checkpoint.urdf (robot description, URDF)
Before this commit: robot robotic_arm, 6 links, 5 joints
Joints:
- joint base_joint: limit lower=-3.14 upper=3.14 -> lower=0 upper=4.71
- joint elbow_joint: axis 1 0 0 -> -1 0 0; limit lower=-2.1 upper=2.1 -> lower=-1.39 upper=1.57
- joint shoulder_joint: axis 1 0 0 -> -1 0 0; limit lower=-1.57 upper=1.57 -> lower=-1.39 upper=1.57
- joint wrist_joint_1: axis 1 0 0 -> -1 0 0; limit lower=-2.1 upper=2.1 -> lower=-1.92 upper=0.7
- joint wrist_joint_2: limit lower=-3.14 upper=3.14 -> lower=-1.92 upper=1.22
